Commit message: new version

File: ZIVID/zivid_description/xacro/pg70_zivid.urdf.xacro (robot description, xacro)
@@ -49,5 +49,5 @@
     </link>
 <!-- LEFT FINGER BASE -->
-    <joint name="${name}_finger_left_joint" type="prismatic" >
+    <joint name="${name}_finger_left_joint" type="fixed" >
       <parent link="${name}_base_link" />
       <child link="${name}_finger_left_link" />
@@ -95,5 +95,5 @@
     </link>
 <!-- RIGHT FINGER BASE -->
-    <joint name="${name}_finger_right_joint" type="prismatic" >
+    <joint name="${name}_finger_right_joint" type="fixed" >
       <mimic joint="${name}_finger_left_joint" multiplier="1" offset="0"/>
       <parent link="${name}_base_link" />
@@ -141,5 +141,5 @@
       <parent link="${name}_base_link" />
       <child link="${name}_object_link" />
-      <origin xyz="0 0 0.21" rpy="0 0 0"/>
+      <origin xyz="0 0 0.16" rpy="0 0 0"/>
    </joint>
     <link name="${name}_object_link">

File: schunk_pg70/urdf/pg70.urdf.xacro (robot description, xacro)
@@ -1,8 +1,116 @@
-<?xml version="1.0" encoding="utf-8"?>
-<robot xmlns:xacro="http://www.ros.org/wiki/xacro"
-  name="schunk_pg70">
-  <xacro:include filename="$(find schunk_pg70)/urdf/pg70_zivid.urdf.xacro"/>
-  <xacro:schunk_pg70 name="schunk_pg70" parent="flange_link" >
-    <origin xyz="-0.04 -0.056 0" rpy="${-pi/2} 0 0" />
-  </xacro:schunk_pg70>
+<?xml version="1.0"?>
+<robot xmlns:xacro="http://www.ros.org/wiki/xacro">
+  <xacro:macro name="schunk_pg70" params="parent name *origin ">
+    <joint name="${name}_base_joint" type="fixed" >
+      <parent link="${parent}" />
+      <child link="${name}_base_link" />
+      <xacro:insert_block name="origin" />
+    </joint>
+<!--     PALM -->
+    <link name="${name}_base_link">
+      <visual>
+        <geometry>
+          <mesh filename="package://schunk_pg70/meshes/pg70.dae" />
+        </geometry>
+        <material name="blue">
+          <color rgba="0 0 1 1"/>
+        </material>
+      </visual>
+      <collision>
+        <geometry>
+          <mesh filename="package://schunk_pg70/meshes/pg70.dae" />
+        </geometry>
+	<material name="blue"/>
+      </collision>
+    </link>
+<!-- LEFT FINGER BASE -->
+    <joint name="${name}_finger_left_joint" type="prismatic" >
+      <parent link="${name}_base_link" />
+      <child link="${name}_finger_left_link" />
+      <limit effort="100" lower="-0.001" upper="0.04" velocity="2.0"/>
+      <origin xyz="0 0 0.0789" rpy="0 0 0"/>
+      <axis xyz="0 1 0" />
+    </joint>
+    <link name="${name}_finger_left_link">
+      <visual>
+        <geometry>
+          <box size="0.03 0.01 0.01"/>
+        </geometry>
+        <material name="black">
+          <color rgba="0 0 0 1"/>
+        </material>
+      </visual>
+      <collision>
+        <geometry>
+          <box size="0.03 0.01 0.01"/>
+        </geometry>
+	<material name="black" />
+      </collision>
+    </link>
+<!-- LEFT FINGERTIP -->
+    <joint name="${name}_fingertip_left_joint" type="fixed" >
+      <parent link="${name}_finger_left_link" />
+      <child link="${name}_fingertip_left_link" />
+      <origin xyz="0 0.01 0.045" rpy="0 0 0"/>
+    </joint>
+    <link name="${name}_fingertip_left_link">
+      <visual>
+        <geometry>
+          <box size="0.03 0.01 0.1"/>
+        </geometry>
+        <material name="silver">
+          <color rgba="0.8 0.8 0.8 1"/>
+        </material>
+      </visual>
+      <collision>
+        <geometry>
+          <box size="0.03 0.01 0.1"/>
+        </geometry>
+	<material name="black"/>
+      </collision>
+    </link>
+<!-- RIGHT FINGER BASE -->
+    <joint name="${name}_finger_right_joint" type="prismatic" >
+      <mimic joint="${name}_finger_left_joint" multiplier="1" offset="0"/>
+      <parent link="${name}_base_link" />
+      <child link="${name}_finger_right_link" />
+      <limit effort="100" lower="-0.001" upper="0.04" velocity="2.0"/>
+      <origin xyz="0 0 0.0789" rpy="-0 0 0"/>
+      <axis xyz="0 -1 0" />
+    </joint>
+    <link name="${name}_finger_right_link">
+      <visual>
+        <geometry>
+          <box size="0.03 0.01 0.01"/>
+        </geometry>
+	<material name="black"/>
+      </visual>
+      <collision>
+        <geometry>
+          <box size="0.03 0.01 0.01"/>
+        </geometry>
+	<material name="black"/>
+      </collision>
+    </link>
+<!-- RIGHT FINGERTIP -->
+    <joint name="${name}_fingertip_right_joint" type="fixed" >
+      <parent link="${name}_finger_right_link" />
+      <child link="${name}_fingertip_right_link" />
+      <origin xyz="0 -0.01 0.045" rpy="0 0 0"/>
+   </joint>
+    <link name="${name}_fingertip_right_link">
+      <visual>
+        <geometry>
+          <box size="0.03 0.01 0.1"/>
+        </geometry>
+	<material name="silver" />
+      </visual>
+      <collision>
+        <geometry>
+          <box size="0.03 0.01 0.1"/>
+        </geometry>
+	<material name="black"/>
+     </collision>
+    </link>
+  </xacro:macro>
 </robot>

File: schunk_pg70/urdf/pg70_visualization.urdf.xacro (robot description, xacro)
@@ -7,6 +7,3 @@
     <origin xyz="0 0 0" rpy="0 0 0" />
   </xacro:schunk_pg70>
-  <xacro:schunk_pg70 name="object" parent="base_link">
-    <origin xyz="0 0 0.2" rpy="0 0 0" />
-  </xacro:schunk_pg70>
  </robot>

Commit message: minor changes

File: ZIVID/zivid_description/xacro/pg70_zivid.urdf.xacro (robot description, xacro)
@@ -141,5 +141,5 @@
       <parent link="${name}_base_link" />
       <child link="${name}_object_link" />
-      <origin xyz="0 0 0.16" rpy="0 0 0"/>
+      <origin xyz="0 0 0.15" rpy="0 0 0"/>
    </joint>
     <link name="${name}_object_link">
